Commit message: workaround ros neotic

File: robotiq_2f_85_gripper_visualization/urdf/robotiq_arg2f_85_macro.xacro (robot description, xacro)
@@ -180,5 +180,5 @@
     </xacro:macro>
     <!-- base link -->
-    <link name="${prefix}base_link"/>
+    <!--<link name="${prefix}base_link"/>-->
     <joint name="${prefix}base_link-${prefix}robotiq_arg2f_base_link" type="fixed">
       <parent link="${prefix}base_link" />
